Commit message: Use TF to calculate positions

File: urdf/edo_gripper_dummy.urdf.xacro (robot description, xacro)
@@ -10,5 +10,5 @@
     <xacro:arg name="robot_name" default="edo"/>
     <xacro:arg name="origin_xyz" default="0 0 0"/>
-    <xacro:arg name="origin_rpy" default="0 0 0"/>
+    <xacro:arg name="origin_rpy" default="0 0 -1.57079632679"/>
     <link name="world"/>
     <gazebo reference="world">
@@ -16,8 +16,8 @@
     </gazebo>
     <xacro:edo hardware_interface="$(arg hardware_interface)" robot_name="$(arg robot_name)" parent="world">
-        <origin xyz="0 0 0" rpy="0 0 0"/>
+        <origin xyz="$(arg origin_xyz)" rpy="$(arg origin_rpy)"/>
     </xacro:edo>
     <xacro:edo_gripper_dummy hardware_interface="$(arg hardware_interface)" robot_name="$(arg robot_name)" parent="$(arg robot_name)_link_ee">
-        <origin xyz="0 0 0" rpy="-${PI / 2} 0 ${PI / 4}"/>
+        <origin xyz="0 0 0" rpy="-${PI / 2} 0 -${PI / 4}"/>
     </xacro:edo_gripper_dummy>
 </robot>

Commit message: Correctly orientate gripper and include griper ee in moveit

File: urdf/edo_gripper_dummy.urdf.xacro (robot description, xacro)
@@ -19,5 +19,5 @@
     </xacro:edo>
     <xacro:edo_gripper_dummy hardware_interface="$(arg hardware_interface)" robot_name="$(arg robot_name)" parent="$(arg robot_name)_link_ee">
-        <origin xyz="0 0 0" rpy="-${PI / 2} 0 -${PI / 4}"/>
+        <origin xyz="0 0 0" rpy="0 0 -${PI / 4}"/>
     </xacro:edo_gripper_dummy>
 </robot>

File: urdf/edo_gripper_dummy.xacro (robot description, xacro)
@@ -25,5 +25,5 @@
             </inertial>
             <visual>
-                <origin xyz="-0.035 0 -0.035" rpy="0 0 0"/>
+                <origin xyz="0 0 0" rpy="0 0 0"/>
                 <geometry>
                     <mesh filename="package://edo_gripper/meshes/base.STL"/>
@@ -32,5 +32,5 @@
             </visual>
             <collision>
-                <origin xyz="-0.035 0 -0.035" rpy="0 0 0"/>
+                <origin xyz="0 0 0" rpy="0 0 0"/>
                 <geometry>
                     <mesh filename="package://edo_gripper/meshes/base.STL"/>
@@ -42,5 +42,5 @@
             <parent link="${robot_name}_gripper_link"/>
             <child link="${robot_name}_gripper_left_base_link"/>
-            <origin xyz="0.025 0.0195 0" rpy="0 0 0"/>
+            <origin xyz="0 0.025 0.0195" rpy="${PI / 2} 0 ${PI / 2}"/>
             <axis xyz="0 0 1"/>
             <limit lower="${-PI / 2}" upper="${PI / 2}"
@@ -114,5 +114,5 @@
             <parent link="${robot_name}_gripper_link"/>
             <child link="${robot_name}_gripper_right_base_link"/>
-            <origin xyz="-0.025 0.0195 0" rpy="${PI} 0 ${PI}"/>
+            <origin xyz="0 -0.025 0.0195" rpy="${PI / 2} 0 -${PI / 2}"/>
             <axis xyz="0 0 1"/>
             <limit lower="${-PI / 2}" upper="${PI / 2}"
@@ -187,5 +187,5 @@
             <parent link="${robot_name}_gripper_link" />
             <child link = "${robot_name}_gripper_link_ee" />
-            <origin xyz="0 0.15 0" rpy="0 0 0" />
+            <origin xyz="0 0 0.125" rpy="0 0 ${PI/4}" />
         </joint>
         <!--  The TCP frame is here defined -->
