Commit message: Temporarily disable gripper control to avoid interference with ros control

File: urdf/edo_gripper_dummy.xacro (robot description, xacro)
@@ -78,7 +78,7 @@
             <parent link="${robot_name}_gripper_left_base_link"/>
             <child link="${robot_name}_gripper_left_finger_link"/>
-            <origin xyz="0 0.04 0" rpy="0 0 ${PI}"/>
-            <axis xyz="0 0 1"/>
-            <limit lower="${-PI*2}" upper="${PI*2}"
+            <origin xyz="0 0.04 0" rpy="0 0 0"/>
+            <axis xyz="0 0 1"/>
+            <limit lower="${-PI / 2}" upper="${PI / 2}"
                    effort="${max_effort}" velocity="${max_velocity}" />
             <dynamics damping="${joint_damping}"/>
@@ -149,12 +149,12 @@
         <joint name="${robot_name}_gripper_right_finger_joint" type="revolute">
             <parent link="${robot_name}_gripper_right_base_link"/>
-            <child link="${robot_name}_gripper_link_finger_right"/>
-            <origin xyz="0 0.04 0" rpy="0 0 ${PI}"/>
-            <axis xyz="0 0 1"/>
-            <limit lower="${-PI*2}" upper="${PI*2}"
-                   effort="${max_effort}" velocity="${max_velocity}" />
-            <dynamics damping="${joint_damping}"/>
-        </joint>
-        <link name="${robot_name}_gripper_link_finger_right">
+            <child link="${robot_name}_gripper_right_finger_link"/>
+            <origin xyz="0 0.04 0" rpy="0 0 0"/>
+            <axis xyz="0 0 1"/>
+            <limit lower="${-PI / 2}" upper="${PI / 2}"
+                   effort="${max_effort}" velocity="${max_velocity}" />
+            <dynamics damping="${joint_damping}"/>
+        </joint>
+        <link name="${robot_name}_gripper_right_finger_link">
             <inertial>
                 <origin xyz="0 0 0" rpy="0 0 0"/>
@@ -196,5 +196,49 @@
                 <robotNamespace>/${robot_name}</robotNamespace>
             </plugin>
-        </gazebo>
+        </gazebo>        <!-- Load Gazebo lib and set the robot namespace -->
+        <transmission name="${robot_name}_gripper_tran_1">
+            <robotNamespace>/${robot_name}</robotNamespace>
+            <type>transmission_interface/SimpleTransmission</type>
+            <joint name="${robot_name}_gripper_left_base_joint">
+                <hardwareInterface>${hardware_interface}</hardwareInterface>
+            </joint>
+            <actuator name="${robot_name}_gripper_motor_1">
+                <hardwareInterface>${hardware_interface}</hardwareInterface>
+                <mechanicalReduction>1</mechanicalReduction>
+            </actuator>
+        </transmission>
+        <transmission name="${robot_name}_gripper_tran_2">
+            <robotNamespace>/${robot_name}</robotNamespace>
+            <type>transmission_interface/SimpleTransmission</type>
+            <joint name="${robot_name}_gripper_right_base_joint">
+                <hardwareInterface>${hardware_interface}</hardwareInterface>
+            </joint>
+            <actuator name="${robot_name}_gripper_motor_2">
+                <hardwareInterface>${hardware_interface}</hardwareInterface>
+                <mechanicalReduction>1</mechanicalReduction>
+            </actuator>
+        </transmission>
+        <transmission name="${robot_name}_gripper_tran_3">
+            <robotNamespace>/${robot_name}</robotNamespace>
+            <type>transmission_interface/SimpleTransmission</type>
+            <joint name="${robot_name}_gripper_left_finger_joint">
+                <hardwareInterface>${hardware_interface}</hardwareInterface>
+            </joint>
+            <actuator name="${robot_name}_gripper_motor_3">
+                <hardwareInterface>${hardware_interface}</hardwareInterface>
+                <mechanicalReduction>1</mechanicalReduction>
+            </actuator>
+        </transmission>
+        <transmission name="${robot_name}_gripper_tran_4">
+            <robotNamespace>/${robot_name}</robotNamespace>
+            <type>transmission_interface/SimpleTransmission</type>
+            <joint name="${robot_name}_gripper_right_finger_joint">
+                <hardwareInterface>${hardware_interface}</hardwareInterface>
+            </joint>
+            <actuator name="${robot_name}_gripper_motor_4">
+                <hardwareInterface>${hardware_interface}</hardwareInterface>
+                <mechanicalReduction>1</mechanicalReduction>
+            </actuator>
+        </transmission>
     </xacro:macro>
 </robot>

Commit message: Remove gazebo plugin and use specific rose node instead

File: urdf/edo_gripper_dummy.xacro (robot description, xacro)
@@ -5,5 +5,5 @@
     <xacro:property name="joint_damping" value="0.5" />
     <xacro:property name="max_effort" value="300"/>
-    <xacro:property name="max_velocity" value="10"/>
+    <xacro:property name="max_velocity" value="0.5"/>
     <xacro:macro name="edo_gripper_dummy" params="parent hardware_interface robot_name *origin">
         <joint name="${robot_name}_gripper_joint" type="fixed">
@@ -187,14 +187,8 @@
             <parent link="${robot_name}_gripper_link" />
             <child link = "${robot_name}_gripper_link_ee" />
-            <origin xyz="0 0 0.08" rpy="0 0 0" />
+            <origin xyz="0 0.15 0" rpy="0 0 0" />
         </joint>
         <!--  The TCP frame is here defined -->
         <link name="${robot_name}_gripper_link_ee"/>
-        <!-- Load Gazebo lib and set the robot namespace -->
-        <gazebo>
-            <plugin name="${robot_name}_gripper" filename="libedo_gripper.so">
-                <robotNamespace>/${robot_name}</robotNamespace>
-            </plugin>
-        </gazebo>        <!-- Load Gazebo lib and set the robot namespace -->
         <transmission name="${robot_name}_gripper_tran_1">
             <robotNamespace>/${robot_name}</robotNamespace>

Commit message: Update pick pose

File: urdf/edo_gripper_dummy.xacro (robot description, xacro)
@@ -187,5 +187,5 @@
             <parent link="${robot_name}_gripper_link" />
             <child link = "${robot_name}_gripper_link_ee" />
-            <origin xyz="0 0 0.125" rpy="0 0 ${PI/4}" />
+            <origin xyz="0 0 0.12" rpy="0 0 ${PI/4}" />
         </joint>
         <!--  The TCP frame is here defined -->

Commit message: Correctly handle robot origin and robot namespace

File: urdf/edo_gripper_dummy.xacro (robot description, xacro)
@@ -6,11 +6,12 @@
     <xacro:property name="max_effort" value="300"/>
     <xacro:property name="max_velocity" value="0.5"/>
+    <xacro:property name="robot_prefix" value="edo"/>
     <xacro:macro name="edo_gripper_dummy" params="parent hardware_interface robot_name *origin">
-        <joint name="${robot_name}_gripper_joint" type="fixed">
+        <joint name="${robot_prefix}_gripper_joint" type="fixed">
             <xacro:insert_block name="origin"/>
             <parent link="${parent}"/>
-            <child link="${robot_name}_gripper_link" />
-        </joint>
-        <link name="${robot_name}_gripper_link">
+            <child link="${robot_prefix}_gripper_link" />
+        </joint>
+        <link name="${robot_prefix}_gripper_link">
             <inertial>
                 <origin xyz="0 0 0" rpy="0 0 0"/>
@@ -39,7 +40,7 @@
             </collision>
         </link>
-        <joint name="${robot_name}_gripper_left_base_joint" type="revolute">
-            <parent link="${robot_name}_gripper_link"/>
-            <child link="${robot_name}_gripper_left_base_link"/>
+        <joint name="${robot_prefix}_gripper_left_base_joint" type="revolute">
+            <parent link="${robot_prefix}_gripper_link"/>
+            <child link="${robot_prefix}_gripper_left_base_link"/>
             <origin xyz="0 0.025 0.0195" rpy="${PI / 2} 0 ${PI / 2}"/>
             <axis xyz="0 0 1"/>
@@ -48,34 +49,34 @@
             <dynamics damping="${joint_damping}"/>
         </joint>
-        <link name="${robot_name}_gripper_left_base_link">
-            <inertial>
-                <origin xyz="0 0 0" rpy="0 0 0"/>
-                <mass value="0.0005"/>
-                <inertia
-                        ixx="1"
-                        ixy="0"
-                        ixz="0"
-                        iyy="1"
-                        iyz="0"
-                        izz="1" />
-            </inertial>
-            <visual>
-                <origin xyz="-0.005 0 -0.04" rpy="0 0 0"/>
-                <geometry>
-                    <mesh filename="package://edo_gripper/meshes/finger_base.STL"/>
-                </geometry>
-                <material name="Brown"/>
-            </visual>
-            <collision>
-                <origin xyz="-0.005 0 -0.04" rpy="0 0 0"/>
-                <geometry>
-                    <mesh filename="package://edo_gripper/meshes/finger_base.STL"/>
-                </geometry>
-                <material name="Brown"/>
-            </collision>
-        </link>
-        <joint name="${robot_name}_gripper_left_finger_joint" type="revolute">
-            <parent link="${robot_name}_gripper_left_base_link"/>
-            <child link="${robot_name}_gripper_left_finger_link"/>
+        <link name="${robot_prefix}_gripper_left_base_link">
+            <inertial>
+                <origin xyz="0 0 0" rpy="0 0 0"/>
+                <mass value="0.0005"/>
+                <inertia
+                        ixx="1"
+                        ixy="0"
+                        ixz="0"
+                        iyy="1"
+                        iyz="0"
+                        izz="1" />
+            </inertial>
+            <visual>
+                <origin xyz="-0.005 0 -0.04" rpy="0 0 0"/>
+                <geometry>
+                    <mesh filename="package://edo_gripper/meshes/finger_base.STL"/>
+                </geometry>
+                <material name="Brown"/>
+            </visual>
+            <collision>
+                <origin xyz="-0.005 0 -0.04" rpy="0 0 0"/>
+                <geometry>
+                    <mesh filename="package://edo_gripper/meshes/finger_base.STL"/>
+                </geometry>
+                <material name="Brown"/>
+            </collision>
+        </link>
+        <joint name="${robot_prefix}_gripper_left_finger_joint" type="revolute">
+            <parent link="${robot_prefix}_gripper_left_base_link"/>
+            <child link="${robot_prefix}_gripper_left_finger_link"/>
             <origin xyz="0 0.04 0" rpy="0 0 0"/>
             <axis xyz="0 0 1"/>
@@ -84,34 +85,34 @@
             <dynamics damping="${joint_damping}"/>
         </joint>
-        <link name="${robot_name}_gripper_left_finger_link">
-            <inertial>
-                <origin xyz="0 0 0" rpy="0 0 0"/>
-                <mass value="0.0005"/>
-                <inertia
-                        ixx="1"
-                        ixy="0"
-                        ixz="0"
-                        iyy="1"
-                        iyz="0"
-                        izz="1" />
-            </inertial>
-            <visual>
-                <origin xyz="-0.071 0 0" rpy="0 0 0"/>
-                <geometry>
-                    <mesh filename="package://edo_gripper/meshes/finger_tip.STL"/>
-                </geometry>
-                <material name="Brown"/>
-            </visual>
-            <collision>
-                <origin xyz="-0.071 0 0" rpy="0 0 0"/>
-                <geometry>
-                    <mesh filename="package://edo_gripper/meshes/finger_tip.STL"/>
-                </geometry>
-                <material name="Brown"/>
-            </collision>
-        </link>
-        <joint name="${robot_name}_gripper_right_base_joint" type="revolute">
-            <parent link="${robot_name}_gripper_link"/>
-            <child link="${robot_name}_gripper_right_base_link"/>
+        <link name="${robot_prefix}_gripper_left_finger_link">
+            <inertial>
+                <origin xyz="0 0 0" rpy="0 0 0"/>
+                <mass value="0.0005"/>
+                <inertia
+                        ixx="1"
+                        ixy="0"
+                        ixz="0"
+                        iyy="1"
+                        iyz="0"
+                        izz="1" />
+            </inertial>
+            <visual>
+                <origin xyz="-0.071 0 0" rpy="0 0 0"/>
+                <geometry>
+                    <mesh filename="package://edo_gripper/meshes/finger_tip.STL"/>
+                </geometry>
+                <material name="Brown"/>
+            </visual>
+            <collision>
+                <origin xyz="-0.071 0 0" rpy="0 0 0"/>
+                <geometry>
+                    <mesh filename="package://edo_gripper/meshes/finger_tip.STL"/>
+                </geometry>
+                <material name="Brown"/>
+            </collision>
+        </link>
+        <joint name="${robot_prefix}_gripper_right_base_joint" type="revolute">
+            <parent link="${robot_prefix}_gripper_link"/>
+            <child link="${robot_prefix}_gripper_right_base_link"/>
             <origin xyz="0 -0.025 0.0195" rpy="${PI / 2} 0 -${PI / 2}"/>
             <axis xyz="0 0 1"/>
@@ -120,34 +121,34 @@
             <dynamics damping="${joint_damping}"/>
         </joint>
-        <link name="${robot_name}_gripper_right_base_link">
-            <inertial>
-                <origin xyz="0 0 0" rpy="0 0 0"/>
-                <mass value="0.0005"/>
-                <inertia
-                        ixx="1"
-                        ixy="0"
-                        ixz="0"
-                        iyy="1"
-                        iyz="0"
-                        izz="1" />
-            </inertial>
-            <visual>
-                <origin xyz="-0.005 0 -0.04" rpy="0 0 0"/>
-                <geometry>
-                    <mesh filename="package://edo_gripper/meshes/finger_base.STL"/>
-                </geometry>
-                <material name="Brown"/>
-            </visual>
-            <collision>
-                <origin xyz="-0.005 0 -0.04" rpy="0 0 0"/>
-                <geometry>
-                    <mesh filename="package://edo_gripper/meshes/finger_base.STL"/>
-                </geometry>
-                <material name="Brown"/>
-            </collision>
-        </link>
-        <joint name="${robot_name}_gripper_right_finger_joint" type="revolute">
-            <parent link="${robot_name}_gripper_right_base_link"/>
-            <child link="${robot_name}_gripper_right_finger_link"/>
+        <link name="${robot_prefix}_gripper_right_base_link">
+            <inertial>
+                <origin xyz="0 0 0" rpy="0 0 0"/>
+                <mass value="0.0005"/>
+                <inertia
+                        ixx="1"
+                        ixy="0"
+                        ixz="0"
+                        iyy="1"
+                        iyz="0"
+                        izz="1" />
+            </inertial>
+            <visual>
+                <origin xyz="-0.005 0 -0.04" rpy="0 0 0"/>
+                <geometry>
+                    <mesh filename="package://edo_gripper/meshes/finger_base.STL"/>
+                </geometry>
+                <material name="Brown"/>
+            </visual>
+            <collision>
+                <origin xyz="-0.005 0 -0.04" rpy="0 0 0"/>
+                <geometry>
+                    <mesh filename="package://edo_gripper/meshes/finger_base.STL"/>
+                </geometry>
+                <material name="Brown"/>
+            </collision>
+        </link>
+        <joint name="${robot_prefix}_gripper_right_finger_joint" type="revolute">
+            <parent link="${robot_prefix}_gripper_right_base_link"/>
+            <child link="${robot_prefix}_gripper_right_finger_link"/>
             <origin xyz="0 0.04 0" rpy="0 0 0"/>
             <axis xyz="0 0 1"/>
@@ -156,5 +157,5 @@
             <dynamics damping="${joint_damping}"/>
         </joint>
-        <link name="${robot_name}_gripper_right_finger_link">
+        <link name="${robot_prefix}_gripper_right_finger_link">
             <inertial>
                 <origin xyz="0 0 0" rpy="0 0 0"/>
@@ -184,11 +185,11 @@
         </link>
         <!--  Here we define another dummy joint. It is placed at the end of the tool, so we can then attach a frame at its TCP for control -->
-        <joint name="${robot_name}_gripper_tip_joint" type="fixed">
-            <parent link="${robot_name}_gripper_link" />
-            <child link = "${robot_name}_gripper_link_ee" />
+        <joint name="${robot_prefix}_gripper_tip_joint" type="fixed">
+            <parent link="${robot_prefix}_gripper_link" />
+            <child link = "${robot_prefix}_gripper_link_ee" />
             <origin xyz="0 0 0.12" rpy="0 0 ${PI/4}" />
         </joint>
         <!--  The TCP frame is here defined -->
-        <link name="${robot_name}_gripper_link_ee"/>
+        <link name="${robot_prefix}_gripper_link_ee"/>
         <gazebo>
             <plugin name="gazebo_grasp_fix" filename="libgazebo_grasp_fix.so">
@@ -196,7 +197,7 @@
                 <arm>
                     <arm_name>robot</arm_name>
-                    <palm_link>${robot_name}_link_6</palm_link>
-                    <gripper_link>${robot_name}_gripper_left_finger_link</gripper_link>
-                    <gripper_link>${robot_name}_gripper_right_finger_link</gripper_link>
+                    <palm_link>${robot_prefix}_link_6</palm_link>
+                    <gripper_link>${robot_prefix}_gripper_left_finger_link</gripper_link>
+                    <gripper_link>${robot_prefix}_gripper_right_finger_link</gripper_link>
                 </arm>
                 <forces_angle_tolerance>0</forces_angle_tolerance>
@@ -209,44 +210,44 @@
             </plugin>
         </gazebo>
-        <transmission name="${robot_name}_gripper_tran_1">
-            <robotNamespace>/${robot_name}</robotNamespace>
-            <type>transmission_interface/SimpleTransmission</type>
-            <joint name="${robot_name}_gripper_left_base_joint">
-                <hardwareInterface>${hardware_interface}</hardwareInterface>
-            </joint>
-            <actuator name="${robot_name}_gripper_motor_1">
-                <hardwareInterface>${hardware_interface}</hardwareInterface>
-                <mechanicalReduction>1</mechanicalReduction>
-            </actuator>
-        </transmission>
-        <transmission name="${robot_name}_gripper_tran_2">
-            <robotNamespace>/${robot_name}</robotNamespace>
-            <type>transmission_interface/SimpleTransmission</type>
-            <joint name="${robot_name}_gripper_right_base_joint">
-                <hardwareInterface>${hardware_interface}</hardwareInterface>
-            </joint>
-            <actuator name="${robot_name}_gripper_motor_2">
-                <hardwareInterface>${hardware_interface}</hardwareInterface>
-                <mechanicalReduction>1</mechanicalReduction>
-            </actuator>
-        </transmission>
-        <transmission name="${robot_name}_gripper_tran_3">
-            <robotNamespace>/${robot_name}</robotNamespace>
-            <type>transmission_interface/SimpleTransmission</type>
-            <joint name="${robot_name}_gripper_left_finger_joint">
-                <hardwareInterface>${hardware_interface}</hardwareInterface>
-            </joint>
-            <actuator name="${robot_name}_gripper_motor_3">
-                <hardwareInterface>${hardware_interface}</hardwareInterface>
-                <mechanicalReduction>1</mechanicalReduction>
-            </actuator>
-        </transmission>
-        <transmission name="${robot_name}_gripper_tran_4">
-            <robotNamespace>/${robot_name}</robotNamespace>
-            <type>transmission_interface/SimpleTransmission</type>
-            <joint name="${robot_name}_gripper_right_finger_joint">
-                <hardwareInterface>${hardware_interface}</hardwareInterface>
-            </joint>
-            <actuator name="${robot_name}_gripper_motor_4">
+        <transmission name="${robot_prefix}_gripper_tran_1">
+            <robotNamespace>/${robot_name}</robotNamespace>
+            <type>transmission_interface/SimpleTransmission</type>
+            <joint name="${robot_prefix}_gripper_left_base_joint">
+                <hardwareInterface>${hardware_interface}</hardwareInterface>
+            </joint>
+            <actuator name="${robot_prefix}_gripper_motor_1">
+                <hardwareInterface>${hardware_interface}</hardwareInterface>
+                <mechanicalReduction>1</mechanicalReduction>
+            </actuator>
+        </transmission>
+        <transmission name="${robot_prefix}_gripper_tran_2">
+            <robotNamespace>/${robot_name}</robotNamespace>
+            <type>transmission_interface/SimpleTransmission</type>
+            <joint name="${robot_prefix}_gripper_right_base_joint">
+                <hardwareInterface>${hardware_interface}</hardwareInterface>
+            </joint>
+            <actuator name="${robot_prefix}_gripper_motor_2">
+                <hardwareInterface>${hardware_interface}</hardwareInterface>
+                <mechanicalReduction>1</mechanicalReduction>
+            </actuator>
+        </transmission>
+        <transmission name="${robot_prefix}_gripper_tran_3">
+            <robotNamespace>/${robot_name}</robotNamespace>
+            <type>transmission_interface/SimpleTransmission</type>
+            <joint name="${robot_prefix}_gripper_left_finger_joint">
+                <hardwareInterface>${hardware_interface}</hardwareInterface>
+            </joint>
+            <actuator name="${robot_prefix}_gripper_motor_3">
+                <hardwareInterface>${hardware_interface}</hardwareInterface>
+                <mechanicalReduction>1</mechanicalReduction>
+            </actuator>
+        </transmission>
+        <transmission name="${robot_prefix}_gripper_tran_4">
+            <robotNamespace>/${robot_name}</robotNamespace>
+            <type>transmission_interface/SimpleTransmission</type>
+            <joint name="${robot_prefix}_gripper_right_finger_joint">
+                <hardwareInterface>${hardware_interface}</hardwareInterface>
+            </joint>
+            <actuator name="${robot_prefix}_gripper_motor_4">
                 <hardwareInterface>${hardware_interface}</hardwareInterface>
                 <mechanicalReduction>1</mechanicalReduction>
